File: cablerouting/dashboard.sch (EAGLE design)
At the start: 30 parts

Commit message: Modeled all low-power-connections in the car.
Parts:
- removed AUX-SOC1, AUX-SOC2, MRTCTRL-SWITCH: 332-02, con-garry:332-02
- removed BRK_CONN1, BRK_LED1, HRN_LED, HRN_LED1, STRB_CONN1: 39-30-02, con-molex-mini-fit:39-30-02
- removed CAN-IGN, CAN-IGN1, CAN-IGN2, CAN-IGN3: 5202-04-N-02, con-ebyelectro:5202-04-N-02
- removed STATE_OUT_CONN1: 39-30-08, con-molex-mini-fit:39-30-08
- added AUX-PACK: AAA, adafruit:AAA
- added BACKUP-LCD-PWR, BAT-AUX, BAT-SIG, BAT-SOC, BRK_LED_OUT, BRK_PDL_IN, DCDC-12V-BUS, DCDC-AUX, DCDC-BMS-SIG, HRN-NOT-LED, MTRCTRL-SWITCH, STRB_IN: 39-30-02, con-molex-mini-fit:39-30-02
- added BAT-CAN-IN, LCD-CAN-IN, LCD-CAN-OUT, MPPT1-CAN-IN, MPPT1-CAN-OUT, MPPT2-CAN-IN, MPPT2-CAN-OUT: 87832-04, con-molex:87832-04
- added BAT-TEMP: 5202-03-N-02, con-ebyelectro:5202-03-N-02
- added DRIVER-CTRL-CAN-IN, DRIVER-CTRL-CAN-OUT, DRIVER-CTRL-TEMP, MTR-CTRL-CAN-IN, MTR-CTRL-CAN-OUT: 43045-04, con-molex-micro-fit:43045-04
- added DRIVER-CTRL-DCDC-EN, DRIVER-CTRL-STRB: 43045-02, con-molex-micro-fit:43045-02
- added MTR-CTRL-CONNECTOR: 43045-14, con-molex-micro-fit:43045-14
- added STATE_IN_CONN1, STATE_OUT_CONN2: 39-30-08, con-molex-mini-fit:39-30-08
- AUX-SOC, AUX-SWITCH, BMS-SWITCH, BTR-SOC, REV-SWITCH: value 332-02 -> 39-30-02; device con-garry:332-02 -> con-molex-mini-fit:39-30-02
Connections:
- new net GND: AUX-PACK.+, AUX-SOC.2, BAT-AUX.2, DC-DC1.1, DCDC-12V-BUS.2, DCDC-AUX.2
- new net N$1: STATE_IN_CONN1.7, STATE_OUT_CONN2.8
- new net N$10: BAT-TEMP-1.1, DRIVER-CTRL-TEMP.1
- new net N$11: DRIVER-CTRL-STRB.1, STRB_IN.1
- new net N$12: MTRCTRL-SWITCH.2
- new net N$13: REV-SWITCH.2
- new net N$2: AUX-PACK.-, AUX-SOC.1, AUX-SWITCH.2
- new net N$3: BMS-SWITCH.2, DCDC-12V-BUS.1
- new net N$4: AUX-SWITCH.1, DCDC-AUX.1
- new net N$5: BAT-AUX.1, BMS-SWITCH.1, DC-DC1.2
- new net N$6: MPPT1-CAN-IN.2, MPPT2-CAN-OUT.1
- new net N$7: DCDC-BMS-SIG.1, DRIVER-CTRL-DCDC-EN.1
- new net N$8: BAT-SOC.1, BTR-SOC.2
- new net N$9: DCDC-BMS-SIG.2, DRIVER-CTRL-DCDC-EN.2
Other:
- moved on the sheet: BACKUP-LCD-1, BACKUP-LCD-2, BACKUP-LCD-3, DASH_IN1, DC-DC1, HD_LED2, HD_LED3, LT_LED3, LT_LED4, LT_LED5, RT_LED3, RT_LED4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
