File: DC-DC/DCDC_combined.sch (EAGLE design)
At the start: 25 parts

Commit message: Revert "Test"
This reverts commit 3d1dbc2c878e3fb79790fd224c3c027493952d56.
Parts:
- removed F2, F3, F6, F8: 4A, f-lf-omniblok-s:SMD-MICRO-FUSE-BLOCK
- removed FUN-OUTPUT-2, FUN-OUTPUT-3, FUN-OUTPUT-4, FUN-OUTPUT-5: 39-30-04, con-molex-mini-fit:39-30-04
- added U$11: VI-JT1-EW, NUSOLAR_Custom:VI-JT1-EW
Connections:
- removed net 12V1: F2.2
- removed net 12V2: F3.2
- removed net 12V3: F6.2
- removed net 12V4: F8.2
- net CAN+: no longer F2.1, F3.1, F6.1, F8.1, FUN-OUTPUT-2.2, FUN-OUTPUT-3.2, FUN-OUTPUT-4.2, FUN-OUTPUT-5.2
- net CAN_H: no longer FUN-OUTPUT-2.4, FUN-OUTPUT-3.4, FUN-OUTPUT-4.4, FUN-OUTPUT-5.4
- net CAN_L: no longer FUN-OUTPUT-2.3, FUN-OUTPUT-3.3, FUN-OUTPUT-4.3, FUN-OUTPUT-5.3
- net GND: no longer FUN-OUTPUT-2.1, FUN-OUTPUT-3.1, FUN-OUTPUT-4.1, FUN-OUTPUT-5.1
