File: lightControl/topshell2_actual.brd (EAGLE design)
At the start: 131.6 x 59.6 mm, 42 parts, among them IC2 74AHC1G08DBV, IC3 74AHC1G08DBV, IC4 74AHC1G32DBV, IC5 74AHC1G32DBV, IC6 REG1117, Q1 PSMN013-30MLC, Q2 PSMN013-30MLC, Q3 PSMN013-30MLC, Q4 PSMN013-30MLC, Q5 PSMN013-30MLC, Q6 PSMN013-30MLC

Commit message: updated_light_control
light control
Parts:
- moved R11 117.6 mm to (118.6, 55.6)
- moved C2 70.1 mm to (70.7, 46.5)
- moved Q1 9.20 mm to (48.6, 57.9), turned to 90 degrees
- moved R4 8.31 mm to (54.8, 58.9), turned to 180 degrees
Routing:
- net N$11: track 68.7 -> 81.7 mm, vias 2 -> 4
- net N$3: track 18.2 -> 30.8 mm
- net N$20: track 24.5 -> 33.3 mm, vias 0 -> 2
- net N$6: track 149.8 -> 157.2 mm
- net N$5: track 6.20 -> 9.22 mm
- net N$14: track 102.6 -> 105.6 mm
- net N$1: track 21.7 -> 23.9 mm
- net N$2: track 5.17 -> 7.00 mm
- net VCC: track 72.4 -> 74.2 mm
- net TS3V555: track 5.79 -> 7.24 mm
- net N$7: track 39.9 -> 41.2 mm
- net VDD: track 48.7 -> 49.7 mm
- net N$8: track 58.7 -> 59.6 mm
- net N$18: track 42.8 -> 43.7 mm
- added copper zone on layer 16, net GND
- added copper zone on layer 1, net NOTGND

Commit message: fixed light board files
ok ay  do kay
Parts:
- removed IC4, IC5: 74AHC1G32DBV, 74xx-little-de:SOT23-5
- added IC1, IC7: 74AHC1G32DBV, 74xx-little-us:SOT23-5
Connections:
- removed net VCC: DASH_IN.6, IC2.5, IC3.5, IC4.5, IC5.5
- net GND: now also IC1.3, IC7.3; no longer IC4.3, IC5.3
- net N$10: now also IC7.4; no longer IC5.4
- net N$11: now also IC7.1; no longer IC5.1
- net N$7: now also IC1.2; no longer IC4.2
- net N$8: now also IC1.1, IC7.2; no longer IC4.1, IC5.2
- net N$9: now also IC1.4; no longer IC4.4
- net VDD: now also DASH_IN.6, IC1.5, IC2.5, IC3.5, IC7.5
Routing:
- net VDD: track 49.7 -> 123.9 mm, vias 1 -> 3
- net VCC: track 74.2 -> 0.00 mm, vias 2 -> 0
- net N$10: track 50.7 -> 0.00 mm, vias 2 -> 0
- net N$9: track 36.1 -> 0.00 mm, vias 2 -> 0
- net N$8: track 59.6 -> 58.3 mm
