File: lightControl/topshell2_actual.sch (EAGLE design)
At the start: 42 parts, among them IC2 74AHC1G08DBV, IC3 74AHC1G08DBV, IC4 74AHC1G32DBV, IC5 74AHC1G32DBV, IC6 REG1117, Q1 PSMN013-30MLC, Q2 PSMN013-30MLC, Q3 PSMN013-30MLC, Q4 PSMN013-30MLC, Q5 PSMN013-30MLC, Q6 PSMN013-30MLC

Commit message: fixed light board files
ok ay  do kay
Parts:
- removed IC4, IC5: 74AHC1G32DBV, 74xx-little-de:74AHC1G32DBV
- added IC1, IC7: 74AHC1G32DBV, 74xx-little-us:74AHC1G32DBV
Connections:
- removed net VCC: DASH_IN.6
- net N$10: now also IC7A.O; no longer IC5A.O
- net N$11: now also IC7A.I0; no longer IC5A.I0
- net N$7: now also IC1A.I1; no longer IC4A.I1
- net N$8: now also IC1A.I0, IC7A.I1; no longer IC4A.I0, IC5A.I1
- net N$9: now also IC1A.O; no longer IC4A.O
- net VDD: now also DASH_IN.6
Other:
- note added: "VDD"
- note removed: "VCC"
