File: Integrated/Integrated_final.brd (EAGLE design)
At the start: 82.5 x 84.8 mm, 24 parts

Commit message: final schematic, just routing now
Parts:
- removed U$7: MCP2515, NUSOLAR_Custom:SO-18W
- added BRK_CONN, BRK_LED, HD_LED, HD_LED1, HRN_LED, HRN_PWR, LT_LED, LT_LED1, LT_LED2, RT_LED, RT_LED1, RT_LED2, STRB_CONN, STRB_LED: 39-30-02?, con-molex-mini-fit:39-30-?02?
- added C1, C2: (no value), SparkFun-Capacitors:0805
- added C12: 2.2uF, eagle-ltspice:C0805
- added C4: 10nF, eagle-ltspice:C0805
- added DASH_IN: 39-30-06?, con-molex-mini-fit:39-30-?06?
- added EXP_TRANS, LOGG_TRANS: MCP2515, NUSOLAR_Custom:SO-18W
- added IC1, IC7: 74AHC1G32DBV, 74xx-little-us:SOT23-5
- added IC2, IC3: 74AHC1G08DBV, 74xx-little-us:SOT23-5
- added IC6: REG1117, burr-brown:SOT223
- added Q1, Q2, Q3, Q4, Q5, Q6: PSMN013-30MLC, transistor-power:LFPAK33
- added R10, R11, R12, R13, R14, R4, R5, R6, R7, R8, R9: 1K, rcl:R0805
- added R2: 220K, rcl:R0805
- added R3: 100K, rcl:R0805
- added SPI_LCD_CONN: FH12-08S-1SH, con-hirose:FH12-08S-1SH
- added TS3V555: LM555D, linear:SO08
- added Y2: (no value), SparkFun-FreqCtrl:HC49US
- moved BREAK/THROTTLE_CONN 151.4 mm to (214.6, 12.7), turned to 90 degrees
- moved R1 126.8 mm to (201.9, 19.1), turned to 0 degrees
- moved CAN_CONN_IN 125.8 mm to (174.0, 21.6)
- moved C3 125.0 mm to (188.0, 67.3)
- moved RGN_BRK_CONN 118.5 mm to (214.6, 24.1), turned to 90 degrees
- moved JP1 117.1 mm to (195.6, 36.8)
- moved C11 117.1 mm to (186.7, 53.3)
- moved C9 117.1 mm to (194.3, 41.9)
- moved JP3 117.1 mm to (200.7, 57.1)
- moved C7 117.1 mm to (221.0, 50.8)
- moved 3_3V_REG 101.2 mm to (154.9, 16.5), turned to 180 degrees
- moved 5V_REG 97.1 mm to (146.1, 16.5), turned to 180 degrees
- moved JP4 94.9 mm to (104.1, 57.1)
- moved CAN_CONN_OUT 69.5 mm to (123.2, 21.6)
- moved JP2 69.3 mm to (91.4, 27.9)
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Connections:
- net A1 renamed A1(LOG)
- net A2 renamed A2(LOG)
- removed net D1: JP5.2
- removed net D9: JP4.8
- new net A0(LOG): JP5.12
- new net A3(LOG): JP5.9
- new net A4(LOG): JP5.8
- new net A5(LOG): JP5.7
- new net CSC: SPI_LCD_CONN.5
- new net D10(LOG): DASH_IN.2, IC1.2, JP4.7, R10.2
- new net D11(LOG): BRK_CONN.1, JP4.6, Q5.4, R9.2
- new net D12(LOG): DASH_IN.5, JP4.5
- new net D13(LOG): JP4.4, Q1.4, R5.2, STRB_CONN.1
- new net D9(LOG): DASH_IN.1, IC1.1, IC7.2, JP4.8, R11.2, R13.2
- new net MISO(LOG): JP5.4
- new net MOSI(LOG): JP5.5
- new net N$10: IC2.2, IC3.1, TS3V555.3
- new net N$15: IC2.4, Q4.4, R7.2
- new net N$16: IC3.4, Q2.4, R8.2
- new net N$17: LT_LED.1, LT_LED1.1, LT_LED2.1, Q4.MB
- new net N$18: Q2.MB, RT_LED.1, RT_LED1.1, RT_LED2.1
- new net N$19: HD_LED.1, HD_LED1.1, Q6.MB
- new net N$24: Q1.MB, STRB_LED.1
- new net N$25: BRK_LED.1, Q5.MB
- new net N$26: Q3.4, R4.2
- new net N$28: IC1.4, IC2.1
- new net N$29: IC3.2, IC7.4
- new net N$3: C2.1, LOGG_TRANS.8, Y2.1
- new net N$30: BRK_LED.2, HD_LED.2, HD_LED1.2, IC6.3, LT_LED.2, LT_LED1.2, LT_LED2.2, RT_LED.2, RT_LED1.2, RT_LED2.2, STRB_LED.2
- new net N$31: HRN_LED.2, HRN_PWR.2
- new net N$32: HRN_LED.1, R14.2
- new net N$33: Q3.MB, R14.1
- new net N$4: SPI_LCD_CONN.2
- new net N$5: SPI_LCD_CONN.3
- new net N$6: C1.2, LOGG_TRANS.7, Y2.2
- new net N$8: R2.1, R3.2, TS3V555.7
- new net N$9: C12.1, R2.2, TS3V555.2, TS3V555.6
- new net PWR: SPI_LCD_CONN.4
- new net SCK(LOG): JP5.6
- new net TS3V555: C4.1, TS3V555.5
- new net VCC: IC1.5, IC2.5, IC3.5, IC7.5
- new net VDD: BRK_CONN.2, DASH_IN.6, IC6.2, R3.1, TS3V555.4, TS3V555.8
- net 3.3V: now also EXP_TRANS.17, EXP_TRANS.18, LOGG_TRANS.17, LOGG_TRANS.18; no longer U$7.17, U$7.18
- net A0: no longer JP5.12
- net A3: no longer JP5.9
- net A4: no longer JP5.8
- net A5: no longer JP5.7
- net CAN_CS: now also EXP_TRANS.16, LOGG_TRANS.16; no longer U$7.16
- net CAN_INT: now also EXP_TRANS.12, LOGG_TRANS.12; no longer U$7.12
- net CAN_RX: now also EXP_TRANS.2, LOGG_TRANS.2; no longer U$7.2
- net CAN_TX: now also EXP_TRANS.1, LOGG_TRANS.1; no longer U$7.1
- net D0: no longer JP5.3
- net D10: no longer JP4.7
- net D11: no longer JP4.6
- net D12: no longer JP4.5
- net D13: no longer JP4.4
- net GND: now also C1.1, C12.2, C2.2, C4.2, EXP_TRANS.9, HRN_PWR.1, IC1.3, IC2.3, IC3.3, IC6.1, IC7.3, LOGG_TRANS.9, Q1.1, Q1.2, Q1.3, Q2.1, Q2.2, Q2.3, Q3.1, Q3.2, Q3.3, Q4.1, Q4.2, Q4.3, Q5.1, Q5.2, Q5.3, Q6.1, Q6.2, Q6.3, R10.1, R11.1, R12.1, R13.1, R4.1, R5.1, R6.1, R7.1, R8.1, R9.1, SPI_LCD_CONN.1, STRB_CONN.2, TS3V555.1; no longer U$7.9
- net MISO: now also EXP_TRANS.15, LOGG_TRANS.15, SPI_LCD_CONN.6; no longer JP5.4, U$7.15
- net MOSI: now also EXP_TRANS.14, LOGG_TRANS.14, SPI_LCD_CONN.8; no longer JP5.5, U$7.14
- net N$1: now also EXP_TRANS.7; no longer U$7.7
- net N$11: now also EXP_TRANS.8; no longer U$7.8
- net RX: now also JP5.3
- net SCK: now also EXP_TRANS.13, LOGG_TRANS.13, SPI_LCD_CONN.7; no longer JP5.6, U$7.13
- net SCL: now also DASH_IN.4, IC7.1, R12.2
- net SDA: now also DASH_IN.3, Q6.4, R6.2
- net TX: now also JP5.2
Routing:
- net 3.3V: track 112.7 -> 31.3 mm, vias 8 -> 2
- net 12V: track 119.3 -> 63.8 mm, vias 2 -> 0
- net 5V: track 53.9 -> 13.3 mm, vias 2 -> 1
- net CAN_H: track 86.4 -> 50.1 mm, vias 4 -> 2
- net CAN_CS: track 28.6 -> 0.00 mm, vias 3 -> 0
- net N$1: track 25.6 -> 0.00 mm
- net N$11: track 24.4 -> 0.00 mm
- net CAN_INT: track 23.5 -> 0.00 mm, vias 2 -> 0
- net MISO: track 21.1 -> 0.00 mm, vias 2 -> 0
- net BRK: track 20.5 -> 0.00 mm
- net THROTTLE: track 20.1 -> 0.00 mm, vias 1 -> 0
- net MOSI: track 19.9 -> 0.00 mm, vias 2 -> 0
- net RGN_BRK: track 18.7 -> 0.00 mm
- net SCK: track 18.6 -> 0.00 mm, vias 2 -> 0
- net CAN_L: track 91.0 -> 72.4 mm, vias 0 -> 2
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Other:
- board size 82.5 x 84.8 mm -> 279.4 x 75.9 mm
