File: Integrated/Integrated_final.sch (EAGLE design)
At the start: 24 parts

Commit message: final schematic, just routing now
Parts:
- removed U$7: MCP2515, NUSOLAR_Custom:MCP2515
- added BRK_CONN, BRK_LED, HD_LED, HD_LED1, HRN_LED, HRN_PWR, LT_LED, LT_LED1, LT_LED2, RT_LED, RT_LED1, RT_LED2, STRB_CONN, STRB_LED: 39-30-02, con-molex-mini-fit:39-30-02
- added C1, C2: (no value), SparkFun-Capacitors:CAP0805
- added C12: 2.2uF, eagle-ltspice:C
- added C4: 10nF, eagle-ltspice:C
- added DASH_IN: 39-30-06, con-molex-mini-fit:39-30-06
- added EXP_TRANS, LOGG_TRANS: MCP2515, NUSOLAR_Custom:MCP2515
- added IC1, IC7: 74AHC1G32DBV, 74xx-little-us:74AHC1G32DBV
- added IC2, IC3: 74AHC1G08DBV, 74xx-little-us:74AHC1G08DBV
- added IC6: REG1117, burr-brown:REG1117
- added Q1, Q2, Q3, Q4, Q5, Q6: PSMN013-30MLC, transistor-power:PSMN013-30MLC
- added R10, R11, R12, R13, R14, R4, R5, R6, R7, R8, R9: 1K, rcl:R-US_R0805
- added R2: 220K, rcl:R-US_R0805
- added R3: 100K, rcl:R-US_R0805
- added SPI_LCD_CONN: FH12-08S-1SH, con-hirose:FH12-08S-1SH
- added TS3V555: LM555D, linear:LM555D
- added Y2: (no value), SparkFun-FreqCtrl:CRYSTALHC49US
Connections:
- net A1 renamed A1(LOG)
- net A2 renamed A2(LOG)
- removed net D1: JP5.2
- removed net D9: JP4.8
- new net A0(LOG): JP5.12
- new net A3(LOG): JP5.9
- new net A4(LOG): JP5.8
- new net A5(LOG): JP5.7
- new net CSC: SPI_LCD_CONN-5.1
- new net D10(LOG): DASH_IN.2, IC1A.I1, JP4.7, R10.2
- new net D11(LOG): BRK_CONN.1, JP4.6, Q5.G, R9.2
- new net D12(LOG): DASH_IN.5, JP4.5
- new net D13(LOG): JP4.4, Q1.G, R5.2, STRB_CONN.1
- new net D9(LOG): DASH_IN.1, IC1A.I0, IC7A.I1, JP4.8, R11.2, R13.2
- new net MISO(LOG): JP5.4
- new net MOSI(LOG): JP5.5
- new net N$10: IC2A.I1, IC3A.I0, TS3V555.Q
- new net N$15: IC2A.O, Q4.G, R7.2
- new net N$16: IC3A.O, Q2.G, R8.2
- new net N$17: LT_LED.1, LT_LED1.1, LT_LED2.1, Q4.D
- new net N$18: Q2.D, RT_LED.1, RT_LED1.1, RT_LED2.1
- new net N$19: HD_LED.1, HD_LED1.1, Q6.D
- new net N$24: Q1.D, STRB_LED.1
- new net N$25: BRK_LED.1, Q5.D
- new net N$26: Q3.G, R4.2
- new net N$28: IC1A.O, IC2A.I0
- new net N$29: IC3A.I1, IC7A.O
- new net N$3: C2.1, LOGG_TRANS.OSC1, Y2.1
- new net N$30: BRK_LED.2, HD_LED.2, HD_LED1.2, IC6.VIN, LT_LED.2, LT_LED1.2, LT_LED2.2, RT_LED.2, RT_LED1.2, RT_LED2.2, STRB_LED.2
- new net N$31: HRN_LED.2, HRN_PWR.2
- new net N$32: HRN_LED.1, R14.2
- new net N$33: Q3.D, R14.1
- new net N$4: SPI_LCD_CONN-2.1
- new net N$5: SPI_LCD_CONN-3.1
- new net N$6: C1.2, LOGG_TRANS.OSC2, Y2.2
- new net N$8: R2.1, R3.2, TS3V555.DIS
- new net N$9: C12.1, R2.2, TS3V555.THR, TS3V555.TR
- new net PWR: SPI_LCD_CONN-4.1
- new net SCK(LOG): JP5.6
- new net TS3V555: C4.1, TS3V555.CV
- new net VDD: BRK_CONN.2, DASH_IN.6, IC6.VOUT, R3.1, TS3V555.R, TS3V555.V+
- net 3.3V: now also EXP_TRANS./RST, EXP_TRANS.VDD, LOGG_TRANS./RST, LOGG_TRANS.VDD; no longer U$7./RST, U$7.VDD
- net A0: no longer JP5.12
- net A3: no longer JP5.9
- net A4: no longer JP5.8
- net A5: no longer JP5.7
- net CAN_CS: now also EXP_TRANS./CS, LOGG_TRANS./CS; no longer U$7./CS
- net CAN_INT: now also EXP_TRANS./INT, LOGG_TRANS./INT; no longer U$7./INT
- net CAN_RX: now also EXP_TRANS.RXCAN, LOGG_TRANS.RXCAN; no longer U$7.RXCAN
- net CAN_TX: now also EXP_TRANS.TXCAN, LOGG_TRANS.TXCAN; no longer U$7.TXCAN
- net D0: no longer JP5.3
- net D10: no longer JP4.7
- net D11: no longer JP4.6
- net D12: no longer JP4.5
- net D13: no longer JP4.4
- net GND: now also C1.1, C12.2, C2.2, C4.2, EXP_TRANS.VSS, HRN_PWR.1, IC6.GND, LOGG_TRANS.VSS, Q1.S, Q2.S, Q3.S, Q4.S, Q5.S, Q6.S, R10.1, R11.1, R12.1, R13.1, R4.1, R5.1, R6.1, R7.1, R8.1, R9.1, SPI_LCD_CONN-1.1, STRB_CONN.2, TS3V555.GND; no longer U$7.VSS
- net MISO: now also EXP_TRANS.SO, LOGG_TRANS.SO, SPI_LCD_CONN-6.1; no longer JP5.4, U$7.SO
- net MOSI: now also EXP_TRANS.SI, LOGG_TRANS.SI, SPI_LCD_CONN-8.1; no longer JP5.5, U$7.SI
- net N$1: now also EXP_TRANS.OSC2; no longer U$7.OSC2
- net N$11: now also EXP_TRANS.OSC1; no longer U$7.OSC1
- net RX: now also JP5.3
- net SCK: now also EXP_TRANS.SCK, LOGG_TRANS.SCK, SPI_LCD_CONN-7.1; no longer JP5.6, U$7.SCK
- net SCL: now also DASH_IN.4, IC7A.I0, R12.2
- net SDA: now also DASH_IN.3, Q6.G, R6.2
- net TX: now also JP5.2
Other:
- note added: "HAZ"
- note added: "HD"
- note added: "HRN"
- note added: "LT"
- note added: "RT"
- note added: "VDD"
- moved on the sheet: 3_3V_REG, 5V_REG, BREAK/THROTTLE_CONN, C10, C11, C3, C5, C6, C7, C8, C9, CAN_CONN_IN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
